File: PIC32MX795F512_DP83848_VS1003_USBHOST/module.sch (EAGLE design)
At the start: 114 parts, among them IC1 IC_USBLC6-2, IC2 LM1117IMPX-3.3, IC3 PIC32MX795F512, IC4 DP83848, IC5 LM1117MPX-2.5, U1 USD-SOCKETUSD, U2 VS1003, X2 CRYSTALS-NOGND-CFPX-217, X3 KUSBVX, Y3 CRYSTAL-GROUNDEDSMD-5X3.2

Commit message: Some updates
Parts:
- added C1: (no value), rcl:C-EUC0402
- added R14: (no value), rcl:R-EU_R0402
- R12: value 0R -> (none)
Connections:
- removed net CE1: R12.2, R13.1, U$2.!CE
- new net SDA1A: IC3.SDA1A/SDI1A/U1ARX/RF2, R14.1, SV1.2
- net 3V: now also C1.1, R12.2, R14.2
- net FLASH_CS: now also IC3.RA1/TCK, R13.1, U$2.!CE; no longer IC3.SDA1A/SDI1A/U1ARX/RF2, R12.1
- net GND: now also C1.2
- net SCL1A: now also R12.1
- net SD_CS: now also IC3.RB15/AN15/CN12/OCFB/; no longer IC3.RA1/TCK
Other:
- moved on the sheet: C11, C38, C6, C7, C8, R12

Commit message: Ethernet AVDD filtering
Parts:
- added C2: (no value), rcl:C-EUC0402
- added L3: (no value), dp_devices:FERRITE-0805
Connections:
- new net A3V: C16.1, C17.1, C21.1, C55.1, C59.1, IC4.ANA33VDD, L3.2, R10.2, R2.2, R3.2, R4.2, R5.2, R7.2, RJ1.P4, RJ1.P5
- net 3V: now also C2.1, L3.1; no longer C16.1, C17.1, C21.1, C55.1, C59.1, IC4.ANA33VDD, R10.2, R2.2, R3.2, R4.2, R5.2, R7.2, RJ1.P4, RJ1.P5
- net GND: now also C2.2
Other:
- moved on the sheet: C1, C11, C3, C38, C4, C6, C7, C8
